File: baumsatz/baumsatz.kicad_sch (KiCad schematic)
At the start: 22 parts, among them J1 ICSP, SW1 SW_SPST, U1 ATtiny85-20S

Commit message: baumsatz update
Parts:
- J1: value ICSP -> Pins_Attiny; footprint footprints:PinHeader -> hacrafu:PinHeader_2x04_Attiny
