File: baumsatz/baumsatz.kicad_pcb (KiCad board)
At the start: 2 copper layers, 88.8 x 98.7 mm, 22 parts, among them J1 ICSP, SW1 SW_SPST, U1 ATtiny85-20S

Commit message: baumsatz update
Parts:
- J1: value ICSP -> Pins_Attiny; footprint footprints:PinHeader -> hacrafu:PinHeader_2x04_Attiny
Routing:
- net /VCC: track 38.1 -> 38.6 mm
- net /RESET: track 31.6 -> 31.1 mm
- net /PB4: track 61.4 -> 60.9 mm
- net /PB2: track 39.1 -> 39.6 mm
- net /GND: vias 80 -> 83

Commit message: bestellung techniktag
Routing:
- net /GND: vias 83 -> 84
Other:
- board text added: "JLCJLCJLCJLC"
Changed lines of the file:
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@@
   (title_block
     (title "Baumsatz")
-    (date "2023-10-08")
+    (date "2023-10-28")
     (company "HaCraFu e.V.")
   )
@@
     (effects (font (size 1.5 1.5) (thickness 0.3)) (justify left))
   )
+  (gr_text "JLCJLCJLCJLC" (at -4.48 64.96) (layer "F.SilkS")
+    (effects (font (size 1 1) (thickness 0.2) bold) (justify left bottom))
+  )
   (gr_text "BAT" (at -4.2 38.2) (layer "F.SilkS")
     (effects (font (size 1.5 1.5) (thickness 0.3)) (justify right))
@@
   (via (at 8.95 49.75) (size 0.8) (drill 0.4) (layers "F.Cu" "B.Cu") (free) (net 17))
   (via (at -8.1 58.7) (size 0.8) (drill 0.4) (layers "F.Cu" "B.Cu") (free) (net 17))
+  (via (at 15.21 23.93) (size 0.8) (drill 0.4) (layers "F.Cu" "B.Cu") (free) (net 17))
   (via (at 2.5 73.4) (size 0.8) (drill 0.4) (layers "F.Cu" "B.Cu") (free) (net 17))
   (via (at 5.6 73.4) (size 0.8) (drill 0.4) (layers "F.Cu" "B.Cu") (free) (net 17))
