File: unicorn_simple/unicorn_simple.kicad_pcb (KiCad board)
At the start: 2 copper layers, 68.8 x 71.1 mm, 7 parts, among them SW1 SW_DIP_x01

Commit message: bestellung techniktag
Parts:
- moved SW1 1.15 mm to (202.7, 110.2)
Routing:
- net VCC: track 129.6 -> 128.8 mm
- net +3V0: track 36.1 -> 35.2 mm
Other:
- board text added: "JLCJLCJLCJLC"
