File: owlthief/owlThief.kicad_pcb (KiCad board)
At the start: 2 copper layers, 82.1 x 94.3 mm, 10 parts, among them Q1 BC 847, SW2 DPDT, T1 Transformer_1P_1S

Commit message: bestellung techniktag
Parts:
- BT1: footprint Battery:BatteryHolder_Keystone_2460_1xAA -> hacrafu:Batteryholder AA SMD 1024
- D1, D2: footprint Binary_Kitchen:5mm_SMD-Pad -> hacrafu:5mm_SMD-Pad
- moved BT1 28.1 mm to (228.4, 115.4)
- moved R1 5.36 mm to (200.5, 98.7)
- moved D1 4.05 mm to (197.9, 64.8)
- moved D2 4.05 mm to (226.1, 64.7)
Routing:
- net Net-(D1-A): track 42.4 -> 52.6 mm
- net /VBAT: track 30.2 -> 34.9 mm
- net Net-(D1-K): track 37.4 -> 41.2 mm
- net Net-(Q1-B): track 13.4 -> 16.3 mm
- net Net-(T1-AA): track 13.4 -> 12.5 mm
- net /3V: track 51.2 -> 50.3 mm
Other:
- board text added: "1"
- board text added: "4"
- board text added: "JLCJLCJLCJLC"
- board text added: "ON OFF"
- board text added: "Owl Thief ${ISSUE_DATE} CC-BY-SA 4.0 Original author: Timo Schindler @blinkyparts.com Mod by: HaCraFu e.V. Martin Müllenhaupt https://hacrafu.de/kits"
- board text added: "green A"
- board text added: "red B"
- board text removed: "CC-BY-SA 4.0"
- board text removed: "Owl Thief"
- board text removed: "Timo Schindler @blinkyparts.com"
- board text removed: "v1.1"

Commit message: fix owlthief?
Parts:
- T1: footprint Binary_Kitchen:SolderWire-0.1sqmm_1x04_P3.6mm_D0.4mm_OD1mm_SMD -> hacrafu:SolderWire-0.1sqmm_1x04_P3.6mm_D0.4mm_OD1mm_SMD
- moved R1 0.05 mm to (200.4, 98.7)
Connections:
- Q1 pad 1: Net-(D1-A) -> Net-(Q1-B)
- Q1 pad 2: Net-(Q1-B) -> GND
- Q1 pad 3: GND -> Net-(D1-A)
Routing:
- net Net-(Q1-B): track 16.3 -> 17.5 mm
- net /VBAT: track 34.9 -> 35.6 mm
Other:
- board text added: "green B"
- board text added: "red A"
- board text removed: "1"
- board text removed: "4"

Commit message: improve owl thief
Connections:
- net /3V renamed Net-(SW2-AB2)
- net /VBAT renamed Net-(BT1-+)
Other:
- board text added: "do not use rechargeable batteries"
Changed lines of the file:
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@@
   (paper "A4")
   (title_block
-    (date "2023-11-11")
+    (date "2024-01-26")
   )
   (layers
@@
   (net 5 "Net-(Q1-B)")
   (net 6 "Net-(T1-AA)")
-  (net 7 "/3V")
+  (net 7 "Net-(BT1-+)")
   (net 8 "unconnected-(SW2-A1-Pad1)")
   (net 9 "unconnected-(SW2-AB1-Pad2)")
   (net 10 "unconnected-(SW2-B1-Pad3)")
   (net 11 "unconnected-(SW2-A2-Pad4)")
-  (net 12 "/VBAT")
+  (net 12 "Net-(SW2-AB2)")
   (footprint "hacrafu:owl" locked (layer "F.Cu")
     (at 224.36 76.663122)
@@
       (net 4 "Net-(D1-A)") (pinfunction "SA") (pintype "passive"))
     (pad "4" smd roundrect (at 7.5 10) (size 4 4) (layers "B.Cu" "B.Paste" "B.Mask") (roundrect_rratio 0.25)
-      (net 7 "/3V") (pinfunction "SB") (pintype "passive"))
+      (net 12 "Net-(SW2-AB2)") (pinfunction "SB") (pintype "passive"))
     (model "${KISYS3DMOD}/Connector_Wire.3dshapes/SolderWire-0.1sqmm_1x04_P3.6mm_D0.4mm_OD1mm.wrl"
       (offset (xyz 0 0 0))
@@
       (stroke (width 0.1) (type solid)) (layer "B.Fab"))
     (pad "1" smd roundrect (at -1.55 0 270) (size 1.3 1.75) (layers "B.Cu" "B.Paste" "B.Mask") (roundrect_rratio 0.1923076923)
-      (net 7 "/3V") (pintype "passive"))
+      (net 12 "Net-(SW2-AB2)") (pintype "passive"))
     (pad "2" smd roundrect (at 1.55 0 270) (size 1.3 1.75) (layers "B.Cu" "B.Paste" "B.Mask") (roundrect_rratio 0.1923076923)
       (net 6 "Net-(T1-AA)") (pintype "passive"))
@@
     (pad "1" smd roundrect (at -31.605 0 180) (size 7.84 6.35) (layers "B.Cu" "B.Paste" "B.Mask") (roundrect_rratio 0)
       (chamfer_ratio 0.4) (chamfer bottom_left)
-      (net 12 "/VBAT") (pinfunction "+") (pintype "passive") (solder_mask_margin 0.102))
+      (net 7 "Net-(BT1-+)") (pinfunction "+") (pintype "passive") (solder_mask_margin 0.102))
     (pad "2" smd roundrect (at 31.605 0 180) (size 7.84 6.35) (layers "B.Cu" "B.Paste" "B.Mask") (roundrect_rratio 0)
       (chamfer_ratio 0.4) (chamfer bottom_right)
@@
       (stroke (width 0.1) (type solid)) (layer "B.Fab"))
     (pad "1" smd rect (at -3.25 -2.5 90) (size 3.15 1.3) (layers "B.Cu" "B.Paste" "B.Mask")
-      (net 8 "unconnected-(SW2-A1-Pad1)") (pinfunction "A1") (pintype "passive"))
+      (net 8 "unconnected-(SW2-A1-Pad1)") (pinfunction "A1") (pintype "passive+no_connect"))
     (pad "2" smd rect (at -3.25 0 90) (size 3.15 1.3) (layers "B.Cu" "B.Paste" "B.Mask")
-      (net 9 "unconnected-(SW2-AB1-Pad2)") (pinfunction "AB1") (pintype "passive"))
+      (net 9 "unconnected-(SW2-AB1-Pad2)") (pinfunction "AB1") (pintype "passive+no_connect"))
     (pad "3" smd rect (at -3.25 2.5 90) (size 3.15 1.3) (layers "B.Cu" "B.Paste" "B.Mask")
-      (net 10 "unconnected-(SW2-B1-Pad3)") (pinfunction "B1") (pintype "passive"))
+      (net 10 "unconnected-(SW2-B1-Pad3)") (pinfunction "B1") (pintype "passive+no_connect"))
     (pad "4" smd rect (at 3.5 -2.5 90) (size 3.15 1.3) (layers "B.Cu" "B.Paste" "B.Mask")
-      (net 11 "unconnected-(SW2-A2-Pad4)") (pinfunction "A2") (pintype "passive"))
+      (net 11 "unconnected-(SW2-A2-Pad4)") (pinfunction "A2") (pintype "passive+no_connect"))
     (pad "5" smd rect (at 3.5 0 90) (size 3.15 1.3) (layers "B.Cu" "B.Paste" "B.Mask")
-      (net 7 "/3V") (pinfunction "AB2") (pintype "passive"))
+      (net 12 "Net-(SW2-AB2)") (pinfunction "AB2") (pintype "passive"))
     (pad "6" smd rect (at 3.5 2.5 90) (size 3.15 1.3) (layers "B.Cu" "B.Paste" "B.Mask")
-      (net 12 "/VBAT") (pinfunction "B2") (pintype "passive"))
+      (net 7 "Net-(BT1-+)") (pinfunction "B2") (pintype "passive"))
     (model "${KICAD6_3DMODEL_DIR}/Connector_PinHeader_2.54mm.3dshapes/PinHeader_2x01_P2.54mm_Vertical_SMD.wrl"
       (offset (xyz 0 0 0))
@@
     (effects (font (size 1.5 1.5) (thickness 0.2)) (justify mirror))
   )
+  (gr_text "do not use \nrechargeable batteries" (at 250.15 106.25) (layer "B.Mask")
+    (effects (font (size 1 1) (thickness 0.2) bold) (justify left bottom mirror))
+  )
   (segment (start 224.61 64.52) (end 224.64 64.55) (width 0.5) (layer "B.Cu") (net 2))
   (segment (start 226.245 81.7825) (end 227.8525 83.39) (width 0.5) (layer "B.Cu") (net 2))
@@
   (segment (start 200.48 100.22) (end 206.97 100.22) (width 0.5) (layer "B.Cu") (net 6))
   (segment (start 206.97 100.22) (end 208.35 101.6) (width 0.5) (layer "B.Cu") (net 6))
-  (segment (start 243.49 88.97) (end 243.49 89.331396) (width 0.5) (layer "B.Cu") (net 7))
-  (segment (start 219.23 101.6) (end 214.74 97.11) (width 0.5) (layer "B.Cu") (net 7))
-  (segment (start 214.74 97.11) (end 200.49 97.11) (width 0.5) (layer "B.Cu") (net 7))
-  (segment (start 223.45 101.6) (end 219.23 101.6) (width 0.5) (layer "B.Cu") (net 7))
-  (segment (start 200.49 97.11) (end 200.45 97.15) (width 0.5) (layer "B.Cu") (net 7))
-  (segment (start 243.49 89.331396) (end 231.221396 101.6) (width 0.5) (layer "B.Cu") (net 7))
-  (segment (start 231.221396 101.6) (end 223.45 101.6) (width 0.5) (layer "B.Cu") (net 7))
-  (segment (start 251.43 91.62) (end 251.43 109.795) (width 0.5) (layer "B.Cu") (net 12))
-  (segment (start 257.075 115.44) (end 259.98 115.44) (width 0.5) (layer "B.Cu") (net 12))
-  (segment (start 245.99 88.97) (end 248.78 88.97) (width 0.5) (layer "B.Cu") (net 12))
-  (segment (start 251.43 109.795) (end 257.075 115.44) (width 0.5) (layer "B.Cu") (net 12))
-  (segment (start 248.78 88.97) (end 251.43 91.62) (width 0.5) (layer "B.Cu") (net 12))
+  (segment (start 251.43 91.62) (end 251.43 109.795) (width 0.5) (layer "B.Cu") (net 7))
+  (segment (start 257.075 115.44) (end 259.98 115.44) (width 0.5) (layer "B.Cu") (net 7))
+  (segment (start 245.99 88.97) (end 248.78 88.97) (width 0.5) (layer "B.Cu") (net 7))
+  (segment (start 251.43 109.795) (end 257.075 115.44) (width 0.5) (layer "B.Cu") (net 7))
+  (segment (start 248.78 88.97) (end 251.43 91.62) (width 0.5) (layer "B.Cu") (net 7))
+  (segment (start 243.49 88.97) (end 243.49 89.331396) (width 0.5) (layer "B.Cu") (net 12))
+  (segment (start 219.23 101.6) (end 214.74 97.11) (width 0.5) (layer "B.Cu") (net 12))
+  (segment (start 214.74 97.11) (end 200.49 97.11) (width 0.5) (layer "B.Cu") (net 12))
+  (segment (start 223.45 101.6) (end 219.23 101.6) (width 0.5) (layer "B.Cu") (net 12))
+  (segment (start 200.49 97.11) (end 200.45 97.15) (width 0.5) (layer "B.Cu") (net 12))
+  (segment (start 243.49 89.331396) (end 231.221396 101.6) (width 0.5) (layer "B.Cu") (net 12))
+  (segment (start 231.221396 101.6) (end 223.45 101.6) (width 0.5) (layer "B.Cu") (net 12))
   (zone (net 1) (net_name "GND") (layer "B.Cu") (hatch edge 0.508)
     (connect_pads (clearance 0.508))
