File: owlthief/owlThief.kicad_sch (KiCad schematic)
At the start: 10 parts, among them Q1 BC 847, SW2 DPDT, T1 Transformer_1P_1S

Commit message: bestellung techniktag
Parts:
- BT1: footprint Battery:BatteryHolder_Keystone_2460_1xAA -> hacrafu:Batteryholder AA SMD 1024
- D1, D2: footprint Binary_Kitchen:5mm_SMD-Pad -> hacrafu:5mm_SMD-Pad
Changed lines of the file:
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@@
       (effects (font (size 1.27 1.27)) (justify left))
     )
-    (property "Footprint" "Battery:BatteryHolder_Keystone_2460_1xAA" (at 27.94 32.766 90)
+    (property "Footprint" "hacrafu:Batteryholder AA SMD 1024" (at 27.94 32.766 90)
       (effects (font (size 1.27 1.27)) hide)
     )
@@
       (effects (font (size 1.27 1.27)))
     )
-    (property "Footprint" "Binary_Kitchen:5mm_SMD-Pad" (at 87.63 107.315 0)
+    (property "Footprint" "hacrafu:5mm_SMD-Pad" (at 87.63 107.315 0)
       (effects (font (size 1.27 1.27)) hide)
     )
@@
       (effects (font (size 1.27 1.27)))
     )
-    (property "Footprint" "Binary_Kitchen:5mm_SMD-Pad" (at 77.47 107.315 0)
+    (property "Footprint" "hacrafu:5mm_SMD-Pad" (at 77.47 107.315 0)
       (effects (font (size 1.27 1.27)) hide)
     )

Commit message: fix owlthief?
Parts:
- Q1: symbol Device:Q_NPN_CBE -> Device:Q_NPN_BEC
- T1: footprint Binary_Kitchen:SolderWire-0.1sqmm_1x04_P3.6mm_D0.4mm_OD1mm_SMD -> hacrafu:SolderWire-0.1sqmm_1x04_P3.6mm_D0.4mm_OD1mm_SMD
Connections:
- net GND: now also Q1.2 (E); no longer Q1.3 (E)
- net at T1.2 (AB): now also Q1.1 (B); no longer Q1.2 (B)
- net at D1.2 (A), T1.3 (SA): now also Q1.3 (C); no longer Q1.1 (C)
Changed lines of the file:
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@@
       (effects (font (size 1.27 1.27)))
     )
-    (property "Footprint" "Binary_Kitchen:SolderWire-0.1sqmm_1x04_P3.6mm_D0.4mm_OD1mm_SMD" (at 60.96 88.265 0)
+    (property "Footprint" "hacrafu:SolderWire-0.1sqmm_1x04_P3.6mm_D0.4mm_OD1mm_SMD" (at 60.96 88.265 0)
       (effects (font (size 1.27 1.27)) hide)
     )
@@
     )
   )
-  (symbol (lib_id "Device:Q_NPN_CBE") (at 68.58 120.015 0) (unit 1)
+  (symbol (lib_id "Device:Q_NPN_BEC") (at 68.58 120.015 0) (unit 1)
     (in_bom yes) (on_board yes) (dnp no)
     (property "Reference" "Q1" (at 73.4314 118.8466 0)

Commit message: improve owl thief
Connections:
- net 3V: no longer names the net of R1.1, SW2.5 (AB2), T1.4 (SB)
- net VBAT: no longer names the net of BT1.1 (+), SW2.6 (B2)
- no-connect marks 0 -> 4
Other:
- moved on the sheet: BT1, SW2
Changed lines of the file:
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@@
   (junction (at 50.8 47.625) (diameter 0) (color 0 0 0 0)
   )
+  (no_connect (at 45.72 57.785))
+  (no_connect (at 35.56 50.165))
+  (no_connect (at 35.56 60.325))
+  (no_connect (at 35.56 55.245))
   (wire (pts (xy 91.44 117.475) (xy 109.22 117.475))
     (stroke (width 0) (type default))
@@
     (stroke (width 0) (type default))
   )
+  (wire (pts (xy 30.861 45.085) (xy 35.56 45.085))
+    (stroke (width 0) (type default))
+  )
   (wire (pts (xy 91.44 130.175) (xy 82.55 130.175))
     (stroke (width 0) (type default))
   )
-  (label "VBAT" (at 27.94 29.21 0) (fields_autoplaced)
-    (effects (font (size 1.27 1.27)) (justify left bottom))
-  )
-  (label "3V" (at 62.865 26.035 180) (fields_autoplaced)
-    (effects (font (size 1.27 1.27)) (justify right bottom))
-  )
-  (label "3V" (at 45.72 47.625 180) (fields_autoplaced)
-    (effects (font (size 1.27 1.27)) (justify right bottom))
-  )
-  (label "VBAT" (at 60.325 36.195 270) (fields_autoplaced)
-    (effects (font (size 1.27 1.27)) (justify right bottom))
-  )
-  (symbol (lib_id "Device:Battery_Cell") (at 27.94 34.29 0) (unit 1)
-    (in_bom yes) (on_board yes) (dnp no)
-    (property "Reference" "BT1" (at 30.9372 31.8516 0)
-      (effects (font (size 1.27 1.27)) (justify left))
-    )
-    (property "Value" "Battery_Cell" (at 30.9372 34.163 0)
-      (effects (font (size 1.27 1.27)) (justify left))
-    )
-    (property "Footprint" "hacrafu:Batteryholder AA SMD 1024" (at 27.94 32.766 90)
-      (effects (font (size 1.27 1.27)) hide)
-    )
-    (property "Datasheet" "~" (at 27.94 32.766 90)
+  (symbol (lib_id "Device:Battery_Cell") (at 30.861 50.165 0) (mirror y) (unit 1)
+    (in_bom yes) (on_board yes) (dnp no)
+    (property "Reference" "BT1" (at 27.8638 47.7266 0)
+      (effects (font (size 1.27 1.27)) (justify left))
+    )
+    (property "Value" "Battery_Cell" (at 27.8638 50.038 0)
+      (effects (font (size 1.27 1.27)) (justify left))
+    )
+    (property "Footprint" "hacrafu:Batteryholder AA SMD 1024" (at 30.861 48.641 90)
+      (effects (font (size 1.27 1.27)) hide)
+    )
+    (property "Datasheet" "~" (at 30.861 48.641 90)
       (effects (font (size 1.27 1.27)) hide)
     )
@@
     )
   )
-  (symbol (lib_id "power:GND") (at 27.94 36.83 0) (unit 1)
-    (in_bom yes) (on_board yes) (dnp no)
-    (property "Reference" "#PWR02" (at 27.94 43.18 0)
-      (effects (font (size 1.27 1.27)) hide)
-    )
-    (property "Value" "GND" (at 28.067 41.2242 0)
-      (effects (font (size 1.27 1.27)))
-    )
-    (property "Footprint" "" (at 27.94 36.83 0)
-      (effects (font (size 1.27 1.27)) hide)
-    )
-    (property "Datasheet" "" (at 27.94 36.83 0)
+  (symbol (lib_id "power:GND") (at 30.861 52.705 0) (mirror y) (unit 1)
+    (in_bom yes) (on_board yes) (dnp no)
+    (property "Reference" "#PWR02" (at 30.861 59.055 0)
+      (effects (font (size 1.27 1.27)) hide)
+    )
+    (property "Value" "GND" (at 30.734 57.0992 0)
+      (effects (font (size 1.27 1.27)))
+    )
+    (property "Footprint" "" (at 30.861 52.705 0)
+      (effects (font (size 1.27 1.27)) hide)
+    )
+    (property "Datasheet" "" (at 30.861 52.705 0)
       (effects (font (size 1.27 1.27)) hide)
     )
@@
     )
   )
-  (symbol (lib_id "hacrafu:DPDT") (at 80.645 32.385 270) (unit 1)
+  (symbol (lib_id "hacrafu:DPDT") (at 39.37 65.405 180) (unit 1)
     (in_bom yes) (on_board yes) (dnp no) (fields_autoplaced)
-    (property "Reference" "SW2" (at 59.182 29.9029 90)
+    (property "Reference" "SW2" (at 41.8521 43.942 90)
       (effects (font (size 1.27 1.27)) (justify right))
     )
-    (property "Value" "DPDT" (at 59.182 32.3271 90)
+    (property "Value" "DPDT" (at 39.4279 43.942 90)
       (effects (font (size 1.27 1.27)) (justify right))
     )
-    (property "Footprint" "hacrafu:Switch_MSS22D18" (at 80.645 32.385 0)
-      (effects (font (size 1.27 1.27)) hide)
-    )
-    (property "Datasheet" "" (at 80.645 32.385 0)
-      (effects (font (size 1.27 1.27)) hide)
-    )
+    (property "Footprint" "hacrafu:Switch_MSS22D18" (at 39.37 65.405 0)
+      (effects (font (size 1.27 1.27)) hide)
+    )
+    (property "Datasheet" "" (at 39.37 65.405 0)
+      (effects (font (size 1.27 1.27)) hide)
+    )
